File: kicad/kicad.sch (KiCad schematic (older format))
At the start: 24 parts, among them SW1 SW_Push, U1 ATmega32U4-AU, Y1 16MHz

Commit message: finished assigning component footprints
Parts:
- MX1, MX2, MX3, MX4: footprint (none) -> MX_Alps_Hybrid:MX-1U-NoLED
- SW1: footprint (none) -> random-keyboard-parts:SKQG-1155865
- USB1: footprint (none) -> random-keyboard-parts:Molex-0548190589
Changed lines of the file:
@@
 F 0 "SW1" H 5200 4135 50  0000 C CNN
 F 1 "SW_Push" H 5200 4044 50  0000 C CNN
-F 2 "" H 5200 4050 50  0001 C CNN
+F 2 "random-keyboard-parts:SKQG-1155865" H 5200 4050 50  0001 C CNN
 F 3 "~" H 5200 4050 50  0001 C CNN
 	1    5200 3850
@@
 F 0 "USB1" V 10587 3267 60  0000 C CNN
 F 1 "Molex-0548190589" V 10481 3267 60  0000 C CNN
-F 2 "" H 10050 3300 60  0001 C CNN
+F 2 "random-keyboard-parts:Molex-0548190589" H 10050 3300 60  0001 C CNN
 F 3 "" H 10050 3300 60  0001 C CNN
 	1    10050 3300
@@
 F 0 "MX1" H 11083 6973 60  0000 C CNN
 F 1 "MX-NoLED" H 11083 6899 20  0000 C CNN
-F 2 "" H 10425 6725 60  0001 C CNN
+F 2 "MX_Alps_Hybrid:MX-1U-NoLED" H 10425 6725 60  0001 C CNN
 F 3 "" H 10425 6725 60  0001 C CNN
 	1    11050 6750
@@
 F 0 "MX3" H 11783 6973 60  0000 C CNN
 F 1 "MX-NoLED" H 11783 6899 20  0000 C CNN
-F 2 "" H 11125 6725 60  0001 C CNN
+F 2 "MX_Alps_Hybrid:MX-1U-NoLED" H 11125 6725 60  0001 C CNN
 F 3 "" H 11125 6725 60  0001 C CNN
 	1    11750 6750
@@
 F 0 "MX2" H 11083 7673 60  0000 C CNN
 F 1 "MX-NoLED" H 11083 7599 20  0000 C CNN
-F 2 "" H 10425 7425 60  0001 C CNN
+F 2 "MX_Alps_Hybrid:MX-1U-NoLED" H 10425 7425 60  0001 C CNN
 F 3 "" H 10425 7425 60  0001 C CNN
 	1    11050 7450
@@
 F 0 "MX4" H 11783 7673 60  0000 C CNN
 F 1 "MX-NoLED" H 11783 7599 20  0000 C CNN
-F 2 "" H 11125 7425 60  0001 C CNN
+F 2 "MX_Alps_Hybrid:MX-1U-NoLED" H 11125 7425 60  0001 C CNN
 F 3 "" H 11125 7425 60  0001 C CNN
 	1    11750 7450
